File: AMS_LTC6813.sch (KiCad schematic (older format))
At the start: 14 parts, among them J1 CELLVOLCON, J2 TEMPSENCON, J3 ISOSPI2, J4 ISOSPI1, U1 LT8631, U2 LTC6813-1

Commit message: 4 archive 10/05/20
Parts:
- added J?: Conn_01x02_Male, symbol Connector:Conn_01x02_Male
- added R? (x2): R, symbol Device:R
- added T? (x2): Transformer_1P_1S, symbol Device:Transformer_1P_1S
- added U? (x2): LTC1380, symbol AMS_custom_lib:LTC1380
- added U?: LTC6255, symbol AMS_custom_lib:LTC6255
Connections:
- net VREG: now also J?.2 (Pin_2), U?.16 (VCC), U?.16 (VCC)
- net ISOMD: now reaches U2.55 (ISOMD)
- net ISOMD: now also J?.1 (Pin_1)
- net IPB: now reaches U2.61 (CSBIMA)
- net IPB: now also U2.64 (IPB), R?.1, T?.1 (AA)
- net IPA: now reaches U2.62 (SCKIPA)
- net IPA: now also R?.1, T?.1 (AA)
- net IMB: now reaches U2.63 (IMB)
- net IMB: now also R?.2, T?.2 (AB)
- net IMB_IN: now reaches J4.4 (IMB_IN)
- net IMB_IN: now also T?.3 (SA)
- net IPB_IN: now reaches J4.5 (IPB_IN)
- net IPB_IN: now also T?.4 (SB)
- net IPA_IN: now reaches J3.1 (IPA_IN)
- net IPA_IN: now also T?.4 (SB)
- net IMA_IN: now reaches J3.2 (IMA_IN)
- net IMA_IN: now also T?.3 (SA)
- new net IMA: R?.2, T?.2 (AB)
- new net VTEMP1: U?.1 (S0)
- new net VTEMP10: U?.2 (S1)
- new net VTEMP11: U?.3 (S2)
- new net VTEMP12: U?.4 (S3)
- new net VTEMP13: U?.5 (S4)
- new net VTEMP14: U?.6 (S5)
- new net VTEMP15: U?.7 (S6)
- new net VTEMP16: U?.8 (S7)
- new net VTEMP2: U?.2 (S1)
- new net VTEMP3: U?.3 (S2)
- new net VTEMP4: U?.4 (S3)
- new net VTEMP5: U?.5 (S4)
- new net VTEMP6: U?.6 (S5)
- new net VTEMP7: U?.7 (S6)
- new net VTEMP8: U?.8 (S7)
- new net VTEMP9: U?.1 (S0)
Other:
- moved on the sheet: U1, U2
