File: _saved_AMS_LTC6813.sch (KiCad schematic (older format))
At the start: 69 parts, among them J1 CELLVOLCON, J10 Conn_01x02_Male, J11 Conn_01x02_Male, J12 Conn_01x02_Male, J13 Conn_01x02_Male, J14 Conn_01x02_Male, J15 Conn_01x02_Male, J16 Conn_01x02_Male, J17 Conn_01x02_Male, J18 Conn_01x02_Male, J19 Conn_01x02_Male, J2 TEMPSENCON, J20 Conn_01x02_Male, J21 Conn_01x02_Male, J22 Conn_01x02_Male, J23 Conn_01x02_Male, J24 Conn_01x02_Male, J25 Conn_01x02_Male, J26 Conn_01x02_Male, J27 Conn_01x02_Male, J28 Conn_01x02_Male, J29 Conn_01x02_Male, J3 ISOSPI2, J30 Conn_01x02_Male, J31 Conn_01x02_Male, J32 Conn_01x02_Male, J33 Conn_01x02_Male, J34 Conn_01x02_Male, J35 Conn_01x02_Male, J36 Conn_01x02_Male, J37 Conn_01x02_Male, J38 Conn_01x02_Male, J39 Conn_01x02_Male, J4 ISOSPI1, J40 Conn_01x02_Male, J41 Conn_01x02_Male, J42 Conn_01x02_Male, J43 Conn_01x02_Male, J44 Conn_01x02_Male, J45 Conn_01x02_Male, J46 Conn_01x02_Male, J47 Conn_01x02_Male, J48 Conn_01x02_Male, J49 Conn_01x02_Male, J5 Conn_01x02_Male, J50 Conn_01x02_Male, J51 Conn_01x02_Male, J52 Conn_01x02_Male, J53 Conn_01x02_Male, J54 Conn_01x02_Male, J55 Conn_01x02_Male, J56 Conn_01x02_Male, J57 Conn_01x02_Male, J58 Conn_01x02_Male, J59 Conn_01x02_Male, J6 Conn_01x02_Male, J60 Conn_01x02_Male, J61 Conn_01x02_Male, J62 Conn_01x02_Male, J63 Conn_01x02_Male, J64 Conn_01x02_Male, J65 Conn_01x02_Male, J66 Conn_01x02_Male, J67 Conn_01x02_Male, J68 Conn_01x02_Male, J7 Conn_01x02_Male, J8 Conn_01x02_Male, J9 Conn_01x02_Male, U2 LTC6813-1

Commit message: working on a newer version
Parts:
- removed J1: CELLVOLCON, AMS_custom_lib:VOLCELLCON, symbol AMS_custom_lib:CELLVOLCON
- removed J2: TEMPSENCON, AMS_custom_lib:TEMPSENSCON, symbol AMS_custom_lib:TEMPSENCON
- removed J3: ISOSPI2, AMS_custom_lib:ISOSPICON, symbol AMS_custom_lib:ISOSPI2
- removed J4: ISOSPI1, AMS_custom_lib:ISOSPICON, symbol AMS_custom_lib:ISOSPI1
Changed lines of the file:
@@
-	1    0    0    -1
-$EndComp
-$Comp
-L AMS_custom_lib:CELLVOLCON J1
-U 1 1 5E4BE5C4
-P 9550 750
-F 0 "J1" H 10328 -54 50  0000 L CNN
-F 1 "CELLVOLCON" H 10328 -145 50  0000 L CNN
-F 2 "AMS_custom_lib:VOLCELLCON" H 9550 750 50  0001 C CNN
-F 3 "" H 9550 750 50  0001 C CNN
-	1    9550 750
-	1    0    0    -1
-$EndComp
-$Comp
-L AMS_custom_lib:ISOSPI1 J4
-U 1 1 5E4BE658
-P 9650 5800
-F 0 "J4" H 10019 5546 50  0000 L CNN
-F 1 "ISOSPI1" H 10019 5455 50  0000 L CNN
-F 2 "AMS_custom_lib:ISOSPICON" H 9650 5800 50  0001 C CNN
-F 3 "" H 9650 5800 50  0001 C CNN
-	1    9650 5800
-	1    0    0    -1
-$EndComp
-$Comp
-L AMS_custom_lib:ISOSPI2 J3
-U 1 1 5E4BE783
-P 9650 5100
-F 0 "J3" H 10019 4846 50  0000 L CNN
-F 1 "ISOSPI2" H 10019 4755 50  0000 L CNN
-F 2 "AMS_custom_lib:ISOSPICON" H 9650 5100 50  0001 C CNN
-F 3 "" H 9650 5100 50  0001 C CNN
-	1    9650 5100
-	1    0    0    -1
-$EndComp
-$Comp
-L AMS_custom_lib:TEMPSENCON J2
-U 1 1 5E4BE857
-P 9600 2650
-F 0 "J2" H 10127 1746 50  0000 L CNN
-F 1 "TEMPSENCON" H 10127 1655 50  0000 L CNN
-F 2 "AMS_custom_lib:TEMPSENSCON" H 9600 2650 50  0001 C CNN
-F 3 "" H 9600 2650 50  0001 C CNN
-	1    9600 2650
 	1    0    0    -1
 $EndComp
@@
 F56 "CELL18" I R 7150 950 50
 $EndSheet
-Text Label 8950 1450 0    50   ~ 0
-GND
-Text Label 8950 2250 0    50   ~ 0
-GND
 Text Label 6000 4400 0    50   ~ 0
 GND
 Wire Wire Line
 	6000 4400 6350 4400
-Wire Wire Line
-	8950 2250 9450 2250
-Wire Wire Line
-	8950 1450 9450 1450
 Text Label 7150 2650 0    50   ~ 0
 CELL1
@@
 Text Label 7150 1550 0    50   ~ 0
 CELL12
-Text Label 9450 850  2    50   ~ 0
-CELL12
-Text Label 9450 950  2    50   ~ 0
-CELL11
-Text Label 9450 1650 2    50   ~ 0
-CELL10
-Text Label 9450 1050 2    50   ~ 0
-CELL9
-Text Label 9450 1150 2    50   ~ 0
-CELL7
-Text Label 9450 1250 2    50   ~ 0
-CELL3
-Text Label 9450 1350 2    50   ~ 0
-CELL1
-Text Label 9450 1550 2    50   ~ 0
-CELL12
-Text Label 9450 1750 2    50   ~ 0
-CELL8
-Text Label 9450 1850 2    50   ~ 0
-CELL6
-Text Label 9450 1950 2    50   ~ 0
-CELL5
-Text Label 9450 2050 2    50   ~ 0
-CELL4
-Text Label 9450 2150 2    50   ~ 0
-CELL2
 Text Label 950  5600 2    50   ~ 0
 V+
@@
 Text Label 1900 5250 1    50   ~ 0
 ICMP
-Text Label 9550 5200 2    50   ~ 0
-IPA_IN
-Text Label 9550 5300 2    50   ~ 0
-IMA_IN
-Text Label 9550 6200 2    50   ~ 0
-IMB_IN
-Text Label 9550 6300 2    50   ~ 0
-IPB_IN
 Text Label 1300 5250 1    50   ~ 0
 IPB
