File: VoltageAndBalanceOneCell.sch (KiCad schematic (older format))
At the start: 5 parts, among them Q1 BSS138

Commit message: working on a newer version
Changed lines of the file:
@@
 AR Path="/5E4D37F6/5E4D5444/5E4D6982" Ref="R50"  Part="1"
 AR Path="/5E4D37F6/5E4D5447/5E4D6982" Ref="R53"  Part="1"
-F 0 "R2" V 3793 1850 50  0000 C CNN
+F 0 "R53" V 3793 1850 50  0000 C CNN
 F 1 "100" V 3884 1850 50  0000 C CNN
 F 2 "Resistor_SMD:R_1206_3216Metric_Pad1.42x1.75mm_HandSolder" V 3930 1850 50  0001 C CNN
@@
 AR Path="/5E4D37F6/5E4D5444/5E4D6989" Ref="R49"  Part="1"
 AR Path="/5E4D37F6/5E4D5447/5E4D6989" Ref="R52"  Part="1"
-F 0 "R1" V 3293 2150 50  0000 C CNN
+F 0 "R52" V 3293 2150 50  0000 C CNN
 F 1 "3.3k" V 3384 2150 50  0000 C CNN
 F 2 "Resistor_THT:R_Axial_DIN0309_L9.0mm_D3.2mm_P15.24mm_Horizontal" V 3430 2150 39  0001 C CNN
@@
 AR Path="/5E4D37F6/5E4D5444/5E4D6990" Ref="C17"  Part="1"
 AR Path="/5E4D37F6/5E4D5447/5E4D6990" Ref="C18"  Part="1"
-F 0 "C1" H 3865 2446 50  0000 L CNN
+F 0 "C18" H 3865 2446 50  0000 L CNN
 F 1 "10n" H 3865 2355 50  0000 L CNN
 F 2 "Resistor_SMD:R_1206_3216Metric_Pad1.42x1.75mm_HandSolder" H 3788 2250 50  0001 C CNN
@@
 AR Path="/5E4D37F6/5E4D5444/5E4D6997" Ref="Q17"  Part="1"
 AR Path="/5E4D37F6/5E4D5447/5E4D6997" Ref="Q18"  Part="1"
-F 0 "Q1" H 4556 2104 50  0000 L CNN
+F 0 "Q18" H 4556 2104 50  0000 L CNN
 F 1 "BSS138" H 4556 2195 50  0000 L CNN
 F 2 "Package_TO_SOT_SMD:SOT-23" H 4550 2075 50  0001 L CIN
@@
 AR Path="/5E4D37F6/5E4D5444/5E4D699E" Ref="R51"  Part="1"
 AR Path="/5E4D37F6/5E4D5447/5E4D699E" Ref="R54"  Part="1"
-F 0 "R3" V 4243 2550 50  0000 C CNN
+F 0 "R54" V 4243 2550 50  0000 C CNN
 F 1 "33" V 4334 2550 50  0000 C CNN
 F 2 "Resistor_SMD:R_1206_3216Metric_Pad1.42x1.75mm_HandSolder" V 4380 2550 50  0001 C CNN

Commit message: adding com
Parts:
- added R55: 33, Resistor_THT:R_Axial_DIN0207_L6.3mm_D2.5mm_P10.16mm_Horizontal, symbol Device:R
- R1: footprint Resistor_THT:R_Axial_DIN0309_L9.0mm_D3.2mm_P15.24mm_Horizontal -> Resistor_SMD:R_1206_3216Metric_Pad1.42x1.75mm_HandSolder
Connections:
- net Cn-1: now also R55.2
- net at Q1.3 (D), R3.1: now also R55.1
Changed lines of the file:
@@
 $Descr A4 11693 8268
 encoding utf-8
-Sheet 3 20
+Sheet 17 20
 Title ""
 Date ""
@@
 AR Path="/5E4D37F6/5E4D5444/5E4D6982" Ref="R50"  Part="1"
 AR Path="/5E4D37F6/5E4D5447/5E4D6982" Ref="R53"  Part="1"
-F 0 "R53" V 3793 1850 50  0000 C CNN
+F 0 "R44" V 3793 1850 50  0000 C CNN
 F 1 "100" V 3884 1850 50  0000 C CNN
 F 2 "Resistor_SMD:R_1206_3216Metric_Pad1.42x1.75mm_HandSolder" V 3930 1850 50  0001 C CNN
@@
 AR Path="/5E4D37F6/5E4D5444/5E4D6989" Ref="R49"  Part="1"
 AR Path="/5E4D37F6/5E4D5447/5E4D6989" Ref="R52"  Part="1"
-F 0 "R52" V 3293 2150 50  0000 C CNN
+F 0 "R43" V 3293 2150 50  0000 C CNN
 F 1 "3.3k" V 3384 2150 50  0000 C CNN
-F 2 "Resistor_THT:R_Axial_DIN0309_L9.0mm_D3.2mm_P15.24mm_Horizontal" V 3430 2150 39  0001 C CNN
+F 2 "Resistor_SMD:R_1206_3216Metric_Pad1.42x1.75mm_HandSolder" V 3430 2150 39  0001 C CNN
 F 3 "~" H 3500 2150 50  0001 C CNN
 	1    3500 2150
@@
 AR Path="/5E4D37F6/5E4D5444/5E4D6990" Ref="C17"  Part="1"
 AR Path="/5E4D37F6/5E4D5447/5E4D6990" Ref="C18"  Part="1"
-F 0 "C18" H 3865 2446 50  0000 L CNN
+F 0 "C15" H 3865 2446 50  0000 L CNN
 F 1 "10n" H 3865 2355 50  0000 L CNN
 F 2 "Resistor_SMD:R_1206_3216Metric_Pad1.42x1.75mm_HandSolder" H 3788 2250 50  0001 C CNN
@@
 AR Path="/5E4D37F6/5E4D5444/5E4D6997" Ref="Q17"  Part="1"
 AR Path="/5E4D37F6/5E4D5447/5E4D6997" Ref="Q18"  Part="1"
-F 0 "Q18" H 4556 2104 50  0000 L CNN
+F 0 "Q15" H 4556 2104 50  0000 L CNN
 F 1 "BSS138" H 4556 2195 50  0000 L CNN
 F 2 "Package_TO_SOT_SMD:SOT-23" H 4550 2075 50  0001 L CIN
@@
 AR Path="/5E4D37F6/5E4D5444/5E4D699E" Ref="R51"  Part="1"
 AR Path="/5E4D37F6/5E4D5447/5E4D699E" Ref="R54"  Part="1"
-F 0 "R54" V 4243 2550 50  0000 C CNN
+F 0 "R45" V 4243 2550 50  0000 C CNN
 F 1 "33" V 4334 2550 50  0000 C CNN
 F 2 "Resistor_SMD:R_1206_3216Metric_Pad1.42x1.75mm_HandSolder" V 4380 2550 50  0001 C CNN
@@
 Wire Wire Line
 	3750 2700 4450 2700
+$Comp
+L Device:R R55
+U 1 1 5F95DD3D
+P 4750 2550
+AR Path="/5E4D37F6/5E4D67CD/5F95DD3D" Ref="R55"  Part="1"
+AR Path="/5E4D37F6/5E4D44D2/5F95DD3D" Ref="R56"  Part="1"
+AR Path="/5E4D37F6/5E4D48B8/5F95DD3D" Ref="R57"  Part="1"
+AR Path="/5E4D37F6/5E4D48BB/5F95DD3D" Ref="R58"  Part="1"
+AR Path="/5E4D37F6/5E4D48BE/5F95DD3D" Ref="R59"  Part="1"
+AR Path="/5E4D37F6/5E4D48C1/5F95DD3D" Ref="R60"  Part="1"
+AR Path="/5E4D37F6/5E4D493D/5F95DD3D" Ref="R61"  Part="1"
+AR Path="/5E4D37F6/5E4D4943/5F95DD3D" Ref="R62"  Part="1"
+AR Path="/5E4D37F6/5E4D494B/5F95DD3D" Ref="R63"  Part="1"
+AR Path="/5E4D37F6/5E4D4954/5F95DD3D" Ref="R64"  Part="1"
+AR Path="/5E4D37F6/5E4D495A/5F95DD3D" Ref="R65"  Part="1"
+AR Path="/5E4D37F6/5E4D495D/5F95DD3D" Ref="R66"  Part="1"
+AR Path="/5E4D37F6/5E4D49AB/5F95DD3D" Ref="R67"  Part="1"
+AR Path="/5E4D37F6/5E4D49AE/5F95DD3D" Ref="R68"  Part="1"
+AR Path="/5E4D37F6/5E4D543E/5F95DD3D" Ref="R69"  Part="1"
+AR Path="/5E4D37F6/5E4D5441/5F95DD3D" Ref="R70"  Part="1"
+AR Path="/5E4D37F6/5E4D5444/5F95DD3D" Ref="R71"  Part="1"
+AR Path="/5E4D37F6/5E4D5447/5F95DD3D" Ref="R72"  Part="1"
+F 0 "R69" H 4820 2596 50  0000 L CNN
+F 1 "33" H 4820 2505 50  0000 L CNN
+F 2 "Resistor_THT:R_Axial_DIN0207_L6.3mm_D2.5mm_P10.16mm_Horizontal" V 4680 2550 50  0001 C CNN
+F 3 "~" H 4750 2550 50  0001 C CNN
+	1    4750 2550
+	1    0    0    -1
+$EndComp
+Wire Wire Line
+	4450 2400 4750 2400
+Connection ~ 4450 2400
+Wire Wire Line
+	4450 2700 4750 2700
+Connection ~ 4450 2700
 $EndSCHEMATC

Commit message: blabl
Changed lines of the file:
@@
 $Descr A4 11693 8268
 encoding utf-8
-Sheet 17 20
+Sheet 3 20
 Title ""
 Date ""
@@
 AR Path="/5E4D37F6/5E4D5444/5E4D6982" Ref="R50"  Part="1"
 AR Path="/5E4D37F6/5E4D5447/5E4D6982" Ref="R53"  Part="1"
-F 0 "R44" V 3793 1850 50  0000 C CNN
+F 0 "R2" V 3793 1850 50  0000 C CNN
 F 1 "100" V 3884 1850 50  0000 C CNN
 F 2 "Resistor_SMD:R_1206_3216Metric_Pad1.42x1.75mm_HandSolder" V 3930 1850 50  0001 C CNN
@@
 AR Path="/5E4D37F6/5E4D5444/5E4D6989" Ref="R49"  Part="1"
 AR Path="/5E4D37F6/5E4D5447/5E4D6989" Ref="R52"  Part="1"
-F 0 "R43" V 3293 2150 50  0000 C CNN
+F 0 "R1" V 3293 2150 50  0000 C CNN
 F 1 "3.3k" V 3384 2150 50  0000 C CNN
 F 2 "Resistor_SMD:R_1206_3216Metric_Pad1.42x1.75mm_HandSolder" V 3430 2150 39  0001 C CNN
@@
 AR Path="/5E4D37F6/5E4D5444/5E4D6990" Ref="C17"  Part="1"
 AR Path="/5E4D37F6/5E4D5447/5E4D6990" Ref="C18"  Part="1"
-F 0 "C15" H 3865 2446 50  0000 L CNN
+F 0 "C1" H 3865 2446 50  0000 L CNN
 F 1 "10n" H 3865 2355 50  0000 L CNN
 F 2 "Resistor_SMD:R_1206_3216Metric_Pad1.42x1.75mm_HandSolder" H 3788 2250 50  0001 C CNN
@@
 AR Path="/5E4D37F6/5E4D5444/5E4D6997" Ref="Q17"  Part="1"
 AR Path="/5E4D37F6/5E4D5447/5E4D6997" Ref="Q18"  Part="1"
-F 0 "Q15" H 4556 2104 50  0000 L CNN
+F 0 "Q1" H 4556 2104 50  0000 L CNN
 F 1 "BSS138" H 4556 2195 50  0000 L CNN
 F 2 "Package_TO_SOT_SMD:SOT-23" H 4550 2075 50  0001 L CIN
@@
 AR Path="/5E4D37F6/5E4D5444/5E4D699E" Ref="R51"  Part="1"
 AR Path="/5E4D37F6/5E4D5447/5E4D699E" Ref="R54"  Part="1"
-F 0 "R45" V 4243 2550 50  0000 C CNN
+F 0 "R3" V 4243 2550 50  0000 C CNN
 F 1 "33" V 4334 2550 50  0000 C CNN
 F 2 "Resistor_SMD:R_1206_3216Metric_Pad1.42x1.75mm_HandSolder" V 4380 2550 50  0001 C CNN
@@
 AR Path="/5E4D37F6/5E4D5444/5F95DD3D" Ref="R71"  Part="1"
 AR Path="/5E4D37F6/5E4D5447/5F95DD3D" Ref="R72"  Part="1"
-F 0 "R69" H 4820 2596 50  0000 L CNN
+F 0 "R55" H 4820 2596 50  0000 L CNN
 F 1 "33" H 4820 2505 50  0000 L CNN
 F 2 "Resistor_THT:R_Axial_DIN0207_L6.3mm_D2.5mm_P10.16mm_Horizontal" V 4680 2550 50  0001 C CNN

Commit message: petite modif
Changed lines of the file:
@@
 AR Path="/5E4D37F6/5E4D5444/5E4D6982" Ref="R50"  Part="1"
 AR Path="/5E4D37F6/5E4D5447/5E4D6982" Ref="R53"  Part="1"
-F 0 "R2" V 3793 1850 50  0000 C CNN
+F 0 "R53" V 3793 1850 50  0000 C CNN
 F 1 "100" V 3884 1850 50  0000 C CNN
 F 2 "Resistor_SMD:R_1206_3216Metric_Pad1.42x1.75mm_HandSolder" V 3930 1850 50  0001 C CNN
@@
 AR Path="/5E4D37F6/5E4D5444/5E4D6989" Ref="R49"  Part="1"
 AR Path="/5E4D37F6/5E4D5447/5E4D6989" Ref="R52"  Part="1"
-F 0 "R1" V 3293 2150 50  0000 C CNN
+F 0 "R52" V 3293 2150 50  0000 C CNN
 F 1 "3.3k" V 3384 2150 50  0000 C CNN
 F 2 "Resistor_SMD:R_1206_3216Metric_Pad1.42x1.75mm_HandSolder" V 3430 2150 39  0001 C CNN
@@
 AR Path="/5E4D37F6/5E4D5444/5E4D6990" Ref="C17"  Part="1"
 AR Path="/5E4D37F6/5E4D5447/5E4D6990" Ref="C18"  Part="1"
-F 0 "C1" H 3865 2446 50  0000 L CNN
+F 0 "C18" H 3865 2446 50  0000 L CNN
 F 1 "10n" H 3865 2355 50  0000 L CNN
 F 2 "Resistor_SMD:R_1206_3216Metric_Pad1.42x1.75mm_HandSolder" H 3788 2250 50  0001 C CNN
@@
 AR Path="/5E4D37F6/5E4D5444/5E4D6997" Ref="Q17"  Part="1"
 AR Path="/5E4D37F6/5E4D5447/5E4D6997" Ref="Q18"  Part="1"
-F 0 "Q1" H 4556 2104 50  0000 L CNN
+F 0 "Q18" H 4556 2104 50  0000 L CNN
 F 1 "BSS138" H 4556 2195 50  0000 L CNN
 F 2 "Package_TO_SOT_SMD:SOT-23" H 4550 2075 50  0001 L CIN
@@
 AR Path="/5E4D37F6/5E4D5444/5E4D699E" Ref="R51"  Part="1"
 AR Path="/5E4D37F6/5E4D5447/5E4D699E" Ref="R54"  Part="1"
-F 0 "R3" V 4243 2550 50  0000 C CNN
+F 0 "R54" V 4243 2550 50  0000 C CNN
 F 1 "33" V 4334 2550 50  0000 C CNN
 F 2 "Resistor_SMD:R_1206_3216Metric_Pad1.42x1.75mm_HandSolder" V 4380 2550 50  0001 C CNN
@@
 AR Path="/5E4D37F6/5E4D5444/5F95DD3D" Ref="R71"  Part="1"
 AR Path="/5E4D37F6/5E4D5447/5F95DD3D" Ref="R72"  Part="1"
-F 0 "R55" H 4820 2596 50  0000 L CNN
+F 0 "R72" H 4820 2596 50  0000 L CNN
 F 1 "33" H 4820 2505 50  0000 L CNN
 F 2 "Resistor_THT:R_Axial_DIN0207_L6.3mm_D2.5mm_P10.16mm_Horizontal" V 4680 2550 50  0001 C CNN

Commit message: tout route sauf voltage channel
Changed lines of the file:
@@
 AR Path="/5E4D37F6/5E4D5444/5E4D6982" Ref="R50"  Part="1"
 AR Path="/5E4D37F6/5E4D5447/5E4D6982" Ref="R53"  Part="1"
-F 0 "R53" V 3793 1850 50  0000 C CNN
+F 0 "R2" V 3793 1850 50  0000 C CNN
 F 1 "100" V 3884 1850 50  0000 C CNN
 F 2 "Resistor_SMD:R_1206_3216Metric_Pad1.42x1.75mm_HandSolder" V 3930 1850 50  0001 C CNN
@@
 AR Path="/5E4D37F6/5E4D5444/5E4D6989" Ref="R49"  Part="1"
 AR Path="/5E4D37F6/5E4D5447/5E4D6989" Ref="R52"  Part="1"
-F 0 "R52" V 3293 2150 50  0000 C CNN
+F 0 "R1" V 3293 2150 50  0000 C CNN
 F 1 "3.3k" V 3384 2150 50  0000 C CNN
 F 2 "Resistor_SMD:R_1206_3216Metric_Pad1.42x1.75mm_HandSolder" V 3430 2150 39  0001 C CNN
@@
 AR Path="/5E4D37F6/5E4D5444/5E4D6990" Ref="C17"  Part="1"
 AR Path="/5E4D37F6/5E4D5447/5E4D6990" Ref="C18"  Part="1"
-F 0 "C18" H 3865 2446 50  0000 L CNN
+F 0 "C1" H 3865 2446 50  0000 L CNN
 F 1 "10n" H 3865 2355 50  0000 L CNN
 F 2 "Resistor_SMD:R_1206_3216Metric_Pad1.42x1.75mm_HandSolder" H 3788 2250 50  0001 C CNN
@@
 AR Path="/5E4D37F6/5E4D5444/5E4D6997" Ref="Q17"  Part="1"
 AR Path="/5E4D37F6/5E4D5447/5E4D6997" Ref="Q18"  Part="1"
-F 0 "Q18" H 4556 2104 50  0000 L CNN
+F 0 "Q1" H 4556 2104 50  0000 L CNN
 F 1 "BSS138" H 4556 2195 50  0000 L CNN
 F 2 "Package_TO_SOT_SMD:SOT-23" H 4550 2075 50  0001 L CIN
@@
 AR Path="/5E4D37F6/5E4D5444/5E4D699E" Ref="R51"  Part="1"
 AR Path="/5E4D37F6/5E4D5447/5E4D699E" Ref="R54"  Part="1"
-F 0 "R54" V 4243 2550 50  0000 C CNN
+F 0 "R3" V 4243 2550 50  0000 C CNN
 F 1 "33" V 4334 2550 50  0000 C CNN
 F 2 "Resistor_SMD:R_1206_3216Metric_Pad1.42x1.75mm_HandSolder" V 4380 2550 50  0001 C CNN
@@
 AR Path="/5E4D37F6/5E4D5444/5F95DD3D" Ref="R71"  Part="1"
 AR Path="/5E4D37F6/5E4D5447/5F95DD3D" Ref="R72"  Part="1"
-F 0 "R72" H 4820 2596 50  0000 L CNN
+F 0 "R55" H 4820 2596 50  0000 L CNN
 F 1 "33" H 4820 2505 50  0000 L CNN
 F 2 "Resistor_THT:R_Axial_DIN0207_L6.3mm_D2.5mm_P10.16mm_Horizontal" V 4680 2550 50  0001 C CNN
