File: AMS_LTC6813.kicad_pcb (KiCad board)
At the start: 2 copper layers, 104.1 x 91.4 mm, 96 parts, among them J1 CELLVOLCON, J2 TEMPSENCON, J3 ISOSPI2, J4 ISOSPI1, Q1 BSS138, Q10 BSS138, Q11 BSS138, Q12 BSS138, Q13 BSS138, Q14 BSS138, Q15 BSS138, Q16 BSS138, Q17 BSS138, Q18 BSS138, Q2 BSS138, Q3 BSS138, Q4 BSS138, Q5 BSS138, Q6 BSS138, Q7 BSS138, Q8 BSS138, Q9 BSS138, U1 LT8631, U2 LTC6813-1

Commit message: working on a newer version
Parts:
- added J10: Conn_01x02_Male, Connector_PinHeader_2.54mm:PinHeader_1x02_P2.54mm_Vertical, F.Cu at (41.0, 66.5)
- added J11: Conn_01x02_Male, Connector_PinHeader_2.54mm:PinHeader_1x02_P2.54mm_Vertical, F.Cu at (41.0, 69.3)
- added J12: Conn_01x02_Male, Connector_PinHeader_2.54mm:PinHeader_1x02_P2.54mm_Vertical, F.Cu at (41.0, 72.0)
- added J13: Conn_01x02_Male, Connector_PinHeader_2.54mm:PinHeader_1x02_P2.54mm_Vertical, F.Cu at (41.0, 74.7)
- added J14: Conn_01x02_Male, Connector_PinHeader_2.54mm:PinHeader_1x02_P2.54mm_Vertical, F.Cu at (41.0, 77.4)
- added J15: Conn_01x02_Male, Connector_PinHeader_2.54mm:PinHeader_1x02_P2.54mm_Vertical, F.Cu at (41.0, 80.1)
- added J16: Conn_01x02_Male, Connector_PinHeader_2.54mm:PinHeader_1x02_P2.54mm_Vertical, F.Cu at (41.0, 82.8)
- added J17: Conn_01x02_Male, Connector_PinHeader_2.54mm:PinHeader_1x02_P2.54mm_Vertical, F.Cu at (41.0, 85.5)
- added J18: Conn_01x02_Male, Connector_PinHeader_2.54mm:PinHeader_1x02_P2.54mm_Vertical, F.Cu at (41.0, 88.2)
- added J19: Conn_01x02_Male, Connector_PinHeader_2.54mm:PinHeader_1x02_P2.54mm_Vertical, F.Cu at (41.0, 90.9)
- added J20: Conn_01x02_Male, Connector_PinHeader_2.54mm:PinHeader_1x02_P2.54mm_Vertical, F.Cu at (41.0, 93.6)
- added J21: Conn_01x02_Male, Connector_PinHeader_2.54mm:PinHeader_1x02_P2.54mm_Vertical, F.Cu at (48.0, 98.0)
- added J22: Conn_01x02_Male, Connector_PinHeader_2.54mm:PinHeader_1x02_P2.54mm_Vertical, F.Cu at (50.7, 98.0)
- added J23: Conn_01x02_Male, Connector_PinHeader_2.54mm:PinHeader_1x02_P2.54mm_Vertical, F.Cu at (53.4, 98.0)
- added J24: Conn_01x02_Male, Connector_PinHeader_2.54mm:PinHeader_1x02_P2.54mm_Vertical, F.Cu at (56.1, 98.0)
- added J25: Conn_01x02_Male, Connector_PinHeader_2.54mm:PinHeader_1x02_P2.54mm_Vertical, F.Cu at (58.8, 98.0)
- added J26: Conn_01x02_Male, Connector_PinHeader_2.54mm:PinHeader_1x02_P2.54mm_Vertical, F.Cu at (61.5, 98.0)
- added J27: Conn_01x02_Male, Connector_PinHeader_2.54mm:PinHeader_1x02_P2.54mm_Vertical, F.Cu at (64.3, 98.0)
- added J28: Conn_01x02_Male, Connector_PinHeader_2.54mm:PinHeader_1x02_P2.54mm_Vertical, F.Cu at (67.0, 98.0)
- added J29: Conn_01x02_Male, Connector_PinHeader_2.54mm:PinHeader_1x02_P2.54mm_Vertical, F.Cu at (69.7, 98.0)
- added J30: Conn_01x02_Male, Connector_PinHeader_2.54mm:PinHeader_1x02_P2.54mm_Vertical, F.Cu at (72.4, 98.0)
- added J31: Conn_01x02_Male, Connector_PinHeader_2.54mm:PinHeader_1x02_P2.54mm_Vertical, F.Cu at (75.1, 98.0)
- added J32: Conn_01x02_Male, Connector_PinHeader_2.54mm:PinHeader_1x02_P2.54mm_Vertical, F.Cu at (77.8, 98.0)
- added J33: Conn_01x02_Male, Connector_PinHeader_2.54mm:PinHeader_1x02_P2.54mm_Vertical, F.Cu at (80.5, 98.0)
- added J34: Conn_01x02_Male, Connector_PinHeader_2.54mm:PinHeader_1x02_P2.54mm_Vertical, F.Cu at (83.2, 98.0)
- added J35: Conn_01x02_Male, Connector_PinHeader_2.54mm:PinHeader_1x02_P2.54mm_Vertical, F.Cu at (85.9, 98.0)
- added J36: Conn_01x02_Male, Connector_PinHeader_2.54mm:PinHeader_1x02_P2.54mm_Vertical, F.Cu at (88.6, 98.0)
- added J37: Conn_01x02_Male, Connector_PinHeader_2.54mm:PinHeader_1x02_P2.54mm_Vertical, F.Cu at (93.0, 93.6)
- added J38: Conn_01x02_Male, Connector_PinHeader_2.54mm:PinHeader_1x02_P2.54mm_Vertical, F.Cu at (93.0, 90.9)
- added J39: Conn_01x02_Male, Connector_PinHeader_2.54mm:PinHeader_1x02_P2.54mm_Vertical, F.Cu at (93.0, 88.2)
- added J40: Conn_01x02_Male, Connector_PinHeader_2.54mm:PinHeader_1x02_P2.54mm_Vertical, F.Cu at (93.0, 85.5)
- added J41: Conn_01x02_Male, Connector_PinHeader_2.54mm:PinHeader_1x02_P2.54mm_Vertical, F.Cu at (93.0, 82.8)
- added J42: Conn_01x02_Male, Connector_PinHeader_2.54mm:PinHeader_1x02_P2.54mm_Vertical, F.Cu at (93.0, 80.1)
- added J43: Conn_01x02_Male, Connector_PinHeader_2.54mm:PinHeader_1x02_P2.54mm_Vertical, F.Cu at (93.0, 77.4)
- added J44: Conn_01x02_Male, Connector_PinHeader_2.54mm:PinHeader_1x02_P2.54mm_Vertical, F.Cu at (93.0, 74.7)
- added J45: Conn_01x02_Male, Connector_PinHeader_2.54mm:PinHeader_1x02_P2.54mm_Vertical, F.Cu at (93.0, 72.0)
- added J46: Conn_01x02_Male, Connector_PinHeader_2.54mm:PinHeader_1x02_P2.54mm_Vertical, F.Cu at (93.0, 69.3)
- added J47: Conn_01x02_Male, Connector_PinHeader_2.54mm:PinHeader_1x02_P2.54mm_Vertical, F.Cu at (93.0, 66.5)
- added J48: Conn_01x02_Male, Connector_PinHeader_2.54mm:PinHeader_1x02_P2.54mm_Vertical, F.Cu at (93.0, 63.8)
- added J49: Conn_01x02_Male, Connector_PinHeader_2.54mm:PinHeader_1x02_P2.54mm_Vertical, F.Cu at (93.0, 61.1)
- added J5: Conn_01x02_Male, Connector_PinHeader_2.54mm:PinHeader_1x02_P2.54mm_Vertical, F.Cu at (41.0, 53.0)
- added J50: Conn_01x02_Male, Connector_PinHeader_2.54mm:PinHeader_1x02_P2.54mm_Vertical, F.Cu at (93.0, 58.4)
- added J51: Conn_01x02_Male, Connector_PinHeader_2.54mm:PinHeader_1x02_P2.54mm_Vertical, F.Cu at (93.0, 55.7)
- added J52: Conn_01x02_Male, Connector_PinHeader_2.54mm:PinHeader_1x02_P2.54mm_Vertical, F.Cu at (93.0, 53.0)
- added J53: Conn_01x02_Male, Connector_PinHeader_2.54mm:PinHeader_1x02_P2.54mm_Vertical, F.Cu at (88.6, 46.0)
- added J54: Conn_01x02_Male, Connector_PinHeader_2.54mm:PinHeader_1x02_P2.54mm_Vertical, F.Cu at (85.9, 46.0)
- added J55: Conn_01x02_Male, Connector_PinHeader_2.54mm:PinHeader_1x02_P2.54mm_Vertical, F.Cu at (83.2, 46.0)
- added J56: Conn_01x02_Male, Connector_PinHeader_2.54mm:PinHeader_1x02_P2.54mm_Vertical, F.Cu at (80.5, 46.0)
- added J57: Conn_01x02_Male, Connector_PinHeader_2.54mm:PinHeader_1x02_P2.54mm_Vertical, F.Cu at (77.8, 46.0)
- added J58: Conn_01x02_Male, Connector_PinHeader_2.54mm:PinHeader_1x02_P2.54mm_Vertical, F.Cu at (75.1, 46.0)
- added J59: Conn_01x02_Male, Connector_PinHeader_2.54mm:PinHeader_1x02_P2.54mm_Vertical, F.Cu at (72.4, 46.0)
- added J6: Conn_01x02_Male, Connector_PinHeader_2.54mm:PinHeader_1x02_P2.54mm_Vertical, F.Cu at (41.0, 55.7)
- added J60: Conn_01x02_Male, Connector_PinHeader_2.54mm:PinHeader_1x02_P2.54mm_Vertical, F.Cu at (69.7, 46.0)
- added J61: Conn_01x02_Male, Connector_PinHeader_2.54mm:PinHeader_1x02_P2.54mm_Vertical, F.Cu at (67.0, 46.0)
- added J62: Conn_01x02_Male, Connector_PinHeader_2.54mm:PinHeader_1x02_P2.54mm_Vertical, F.Cu at (64.3, 46.0)
- added J63: Conn_01x02_Male, Connector_PinHeader_2.54mm:PinHeader_1x02_P2.54mm_Vertical, F.Cu at (61.5, 46.0)
- added J64: Conn_01x02_Male, Connector_PinHeader_2.54mm:PinHeader_1x02_P2.54mm_Vertical, F.Cu at (58.8, 46.0)
- added J65: Conn_01x02_Male, Connector_PinHeader_2.54mm:PinHeader_1x02_P2.54mm_Vertical, F.Cu at (56.1, 46.0)
- added J66: Conn_01x02_Male, Connector_PinHeader_2.54mm:PinHeader_1x02_P2.54mm_Vertical, F.Cu at (53.4, 46.0)
- added J67: Conn_01x02_Male, Connector_PinHeader_2.54mm:PinHeader_1x02_P2.54mm_Vertical, F.Cu at (50.7, 46.0)
- added J68: Conn_01x02_Male, Connector_PinHeader_2.54mm:PinHeader_1x02_P2.54mm_Vertical, F.Cu at (48.0, 46.0)
- added J7: Conn_01x02_Male, Connector_PinHeader_2.54mm:PinHeader_1x02_P2.54mm_Vertical, F.Cu at (41.0, 58.4)
- added J8: Conn_01x02_Male, Connector_PinHeader_2.54mm:PinHeader_1x02_P2.54mm_Vertical, F.Cu at (41.0, 61.1)
- added J9: Conn_01x02_Male, Connector_PinHeader_2.54mm:PinHeader_1x02_P2.54mm_Vertical, F.Cu at (41.0, 63.8)
- moved J1 117.0 mm to (149.0, 131.0)
- moved C11 107.6 mm to (295.3, 107.0)
- moved C3 107.6 mm to (286.2, 147.7)
- moved C5 107.6 mm to (286.2, 134.1)
- moved C6 107.6 mm to (264.4, 147.7)
- moved R11 107.6 mm to (264.4, 161.2)
- moved R13 107.6 mm to (274.9, 131.1)
- moved R21 107.6 mm to (295.3, 120.6)
- moved R24 107.6 mm to (264.4, 134.1)
- moved R36 107.6 mm to (268.6, 120.6)
- moved R4 107.6 mm to (274.9, 158.2)
- moved R44 107.6 mm to (268.6, 107.0)
- moved R5 107.6 mm to (286.2, 161.2)
- moved R7 107.6 mm to (274.9, 144.6)
- moved Q10 107.6 mm to (188.5, 140.8)
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Connections:
- net Net-(J3-Pad1) renamed /IPA_IN
- net Net-(J3-Pad2) renamed /IMA_IN
- net Net-(J4-Pad4) renamed /IMB_IN
- net Net-(J4-Pad5) renamed /IPB_IN
- U2 pad 1: /C18 -> /V+
- U2 pad 38: /GND -> /C0
- U2 pad 39: Net-(U2-Pad39) -> /GPIO1
- U2 pad 40: Net-(U2-Pad40) -> /GPIO2
- U2 pad 41: Net-(U2-Pad41) -> /GPIO3
- U2 pad 42: Net-(U2-Pad42) -> /GPIO4
- U2 pad 43: Net-(U2-Pad43) -> /GPIO5
- U2 pad 44: Net-(U2-Pad44) -> /GPIO6
- U2 pad 45: Net-(U2-Pad45) -> /GPIO7
- U2 pad 46: Net-(U2-Pad46) -> /GPIO8
- U2 pad 47: Net-(U2-Pad47) -> /GPIO9
- U2 pad 48: Net-(U2-Pad48) -> /VREG
- U2 pad 49: Net-(U2-Pad49) -> /DRIVE
- U2 pad 50: Net-(U2-Pad50) -> /VREF2
- U2 pad 51: Net-(U2-Pad51) -> /VREF1
- U2 pad 52: Net-(U2-Pad52) -> /DTEN
- U2 pad 53: Net-(U2-Pad53) -> /SDI
- U2 pad 54: Net-(U2-Pad54) -> /SDO
- U2 pad 55: Net-(U2-Pad55) -> /ISOMD
- U2 pad 56: Net-(U2-Pad56) -> /WDT
- U2 pad 57: Net-(U2-Pad57) -> /IBIAS
- U2 pad 58: Net-(U2-Pad58) -> /ICMP
- U2 pad 59: Net-(U2-Pad59) -> /V-
- U2 pad 60: Net-(U2-Pad60) -> /V-
- U2 pad 61: Net-(U2-Pad61) -> /CSBIMA
- U2 pad 62: Net-(U2-Pad62) -> /SCKIPA
- U2 pad 63: Net-(U2-Pad63) -> /IMB
- U2 pad 64: Net-(U2-Pad64) -> /IPB
Routing:
- net /V-: track 0.00 -> 51.3 mm
- net /C18: track 2.72 -> 32.0 mm
- net /DRIVE: track 0.00 -> 28.5 mm
- net /C11: track 0.00 -> 28.5 mm
- net /S3: track 0.00 -> 28.4 mm
- net /C3: track 0.00 -> 28.4 mm
- net /V+: track 0.00 -> 28.4 mm
- net /IPB: track 0.00 -> 28.4 mm
- net /VREG: track 0.00 -> 28.4 mm
- net /S11: track 0.00 -> 28.4 mm
- net /VREF2: track 0.00 -> 27.5 mm
- net /S12: track 0.00 -> 27.5 mm
- net /S4: track 0.00 -> 27.5 mm
- net /C2: track 0.00 -> 27.5 mm
- net /IMB: track 0.00 -> 27.5 mm
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Other:
- board outline removed
- board text added: "IPB IMB SCK IPA CSB IMA V- V- ICMP IBIAS WDT ISOMD SDO SDI DTEN VREF1 VREF2 DRIVE"
- board text added: "S11 C10 S10 C9 S9 C8 S8 C7 S7 C6 S6 C5 S5 C4 S4 C3"
- board text added: "V+ C18 S18 C17 S17 C16 S16 C15 S15 C14 S14 C13 S13 C12 S12 C11"
- board text added: "VREG GPIO9 GPIO8 GPIO7 GPIO6 GPIO5 GPIO4 GPIO3 GPIO2 GPIO1 C0 S1 C1 S2 C2 S3"

Commit message: blabl
Parts:
- added J69: Conn_02x02_Counter_Clockwise, Connector_PinHeader_2.54mm:PinHeader_2x02_P2.54mm_Vertical, F.Cu at (171.2, 13.8)
- added J70: Conn_01x03_Female, Connector_PinHeader_2.54mm:PinHeader_1x03_P2.54mm_Vertical, F.Cu at (167.5, 13.8)
- added J71: Conn_02x20_Counter_Clockwise, Connector_IDC:IDC-Header_2x20_P2.54mm_Vertical, F.Cu at (159.7, 17.7)
- added R55: 33, Resistor_THT:R_Axial_DIN0207_L6.3mm_D2.5mm_P10.16mm_Horizontal, F.Cu at (268.5, 13.5)
- added R56: 33, Resistor_THT:R_Axial_DIN0207_L6.3mm_D2.5mm_P10.16mm_Horizontal, F.Cu at (284.6, 55.2)
- added R57: 33, Resistor_THT:R_Axial_DIN0207_L6.3mm_D2.5mm_P10.16mm_Horizontal, F.Cu at (254.0, 77.5)
- added R58: 33, Resistor_THT:R_Axial_DIN0207_L6.3mm_D2.5mm_P10.16mm_Horizontal, F.Cu at (268.5, 65.6)
- added R59: 33, Resistor_THT:R_Axial_DIN0207_L6.3mm_D2.5mm_P10.16mm_Horizontal, F.Cu at (284.6, 44.8)
- added R60: 33, Resistor_THT:R_Axial_DIN0207_L6.3mm_D2.5mm_P10.16mm_Horizontal, F.Cu at (268.5, 55.2)
- added R61: 33, Resistor_THT:R_Axial_DIN0207_L6.3mm_D2.5mm_P10.16mm_Horizontal, F.Cu at (237.9, 77.5)
- added R62: 33, Resistor_THT:R_Axial_DIN0207_L6.3mm_D2.5mm_P10.16mm_Horizontal, F.Cu at (284.6, 34.4)
- added R63: 33, Resistor_THT:R_Axial_DIN0207_L6.3mm_D2.5mm_P10.16mm_Horizontal, F.Cu at (268.5, 44.8)
- added R64: 33, Resistor_THT:R_Axial_DIN0207_L6.3mm_D2.5mm_P10.16mm_Horizontal, F.Cu at (157.1, 77.5)
- added R65: 33, Resistor_THT:R_Axial_DIN0207_L6.3mm_D2.5mm_P10.16mm_Horizontal, F.Cu at (284.6, 23.9)
- added R66: 33, Resistor_THT:R_Axial_DIN0207_L6.3mm_D2.5mm_P10.16mm_Horizontal, F.Cu at (221.7, 77.5)
- added R67: 33, Resistor_THT:R_Axial_DIN0207_L6.3mm_D2.5mm_P10.16mm_Horizontal, F.Cu at (268.5, 34.4)
- added R68: 33, Resistor_THT:R_Axial_DIN0207_L6.3mm_D2.5mm_P10.16mm_Horizontal, F.Cu at (205.6, 77.5)
- added R69: 33, Resistor_THT:R_Axial_DIN0207_L6.3mm_D2.5mm_P10.16mm_Horizontal, F.Cu at (284.6, 13.5)
- added R70: 33, Resistor_THT:R_Axial_DIN0207_L6.3mm_D2.5mm_P10.16mm_Horizontal, F.Cu at (189.4, 77.5)
- added R71: 33, Resistor_THT:R_Axial_DIN0207_L6.3mm_D2.5mm_P10.16mm_Horizontal, F.Cu at (268.5, 23.9)
- added R72: 33, Resistor_THT:R_Axial_DIN0207_L6.3mm_D2.5mm_P10.16mm_Horizontal, F.Cu at (173.2, 77.5)
- added R73: 100, Resistor_SMD:R_1206_3216Metric_Pad1.42x1.75mm_HandSolder, F.Cu at (183.0, 13.1)
- added R74: 5k, Resistor_SMD:R_1206_3216Metric_Pad1.42x1.75mm_HandSolder, F.Cu at (178.0, 13.1)
- J1: value CELLVOLCON -> Conn_01x06; footprint AMS_custom_lib:VOLCELLCON -> Connector_PinHeader_2.54mm:PinHeader_1x06_P2.54mm_Vertical
- J2: value TEMPSENCON -> Conn_01x03_Female; footprint AMS_custom_lib:TEMPSENSCON -> Connector_PinHeader_2.54mm:PinHeader_1x03_P2.54mm_Vertical
- J3: value ISOSPI2 -> Conn_01x06; footprint AMS_custom_lib:ISOSPICON -> Connector_PinHeader_2.54mm:PinHeader_1x06_P2.54mm_Horizontal
- J4: value ISOSPI1 -> Conn_02x02_Counter_Clockwise; footprint AMS_custom_lib:ISOSPICON -> Connector_PinHeader_2.54mm:PinHeader_2x02_P2.54mm_Vertical
- R1, R10, R13, R16, R19, R22, R25, R28, R31, R34, R37, R4, R40, R43, R46, R49, R52, R7: footprint Resistor_THT:R_Axial_DIN0309_L9.0mm_D3.2mm_P15.24mm_Horizontal -> Resistor_SMD:R_1206_3216Metric_Pad1.42x1.75mm_HandSolder
- U1: value LT8631 -> LTC6820; footprint Package_SO:TSSOP-20_4.4x6.5mm_P0.65mm -> Package_SO:MSOP-16_3x4mm_P0.5mm
Connections:
- net /VoltageMeasurementsAndBalancing/CELL13 renamed /CELL13
- net /VoltageMeasurementsAndBalancing/CELL14 renamed /CELL14
- net /VoltageMeasurementsAndBalancing/CELL15 renamed /CELL15
- net /VoltageMeasurementsAndBalancing/CELL16 renamed /CELL16
- net /VoltageMeasurementsAndBalancing/CELL17 renamed /CELL17
- net /VoltageMeasurementsAndBalancing/CELL18 renamed /CELL18
- net Net-(J2-Pad2) renamed /ICMB
- net Net-(U1-Pad15) renamed /ICMP1
- net Net-(U1-Pad4) renamed /SCK
- C15 pad 2: /GND -> /C0
- J1 pad 1: /CELL12 -> /VDD1
- J1 pad 2: /CELL11 -> /C0
- J1 pad 3: /CELL9 -> /MOSI
- J1 pad 4: /CELL7 -> /MISO
- J1 pad 5: /CELL3 -> /CS
- J1 pad 6: /CELL1 -> /SCk
- J2 pad 1: Net-(J2-Pad1) -> /IBIAS
- J2 pad 3: Net-(J2-Pad3) -> /C0
- J3 pad 1: /IPA_IN -> /SCKIPA1
- J3 pad 2: /IMA_IN -> /CSBIMA1
- J3 pad 3: Net-(J3-Pad3) -> /SDO
- J3 pad 4: Net-(J3-Pad4) -> /SDI
- J3 pad 5: Net-(J3-Pad5) -> /C0
- J4 pad 1: Net-(J4-Pad1) -> /SCKIPA
- J4 pad 2: Net-(J4-Pad2) -> /CSBIMA
- J4 pad 3: Net-(J4-Pad3) -> /IM
- J4 pad 4: /IMB_IN -> /IP
- J63 pad 1: /V- -> /C0
- J63 pad 2: /V- -> /C0
- J64 pad 1: /V- -> /C0
- J64 pad 2: /V- -> /C0
- R45 pad 2: /GND -> /C0
- U1 pad 10: Net-(U1-Pad10) -> /IM
- U1 pad 11: Net-(U1-Pad11) -> /IP
- U1 pad 12: Net-(U1-Pad12) -> /VDD1
- U1 pad 14: Net-(U1-Pad14) -> /C0
- U1 pad 16: Net-(U1-Pad16) -> /IBIAS1
- U1 pad 2: Net-(U1-Pad2) -> /MOSI
- U1 pad 3: Net-(U1-Pad3) -> /MISO
- U1 pad 5: Net-(U1-Pad5) -> /CS
- U1 pad 6: Net-(U1-Pad6) -> /VDD1
- U1 pad 7: Net-(U1-Pad7) -> /VDD1
- U1 pad 8: Net-(U1-Pad8) -> /VDD1
- U1 pad 9: Net-(U1-Pad9) -> /VDD1
- U2 pad 59: /V- -> /C0
- U2 pad 60: /V- -> /C0
Routing:
- net /C0: track 23.9 -> 75.2 mm
- net /V-: track 51.3 -> 0.00 mm

Commit message: petite modif
Parts:
- added C19: 1u, Capacitor_SMD:C_1210_3225Metric_Pad1.42x2.65mm_HandSolder, F.Cu at (101.5, 168.0)
- added C20: 1u, Capacitor_SMD:C_1210_3225Metric_Pad1.42x2.65mm_HandSolder, F.Cu at (78.7, 173.2)
- added C21: 1u, Capacitor_SMD:C_1210_3225Metric_Pad1.42x2.65mm_HandSolder, F.Cu at (78.7, 170.0)
- added C22: 0.1u, Capacitor_SMD:C_1210_3225Metric_Pad1.42x2.65mm_HandSolder, F.Cu at (83.7, 170.0)
- added J72: Conn_01x02_Male, Connector_PinHeader_2.54mm:PinHeader_1x02_P2.54mm_Vertical, F.Cu at (64.0, 119.0)
- added J73: Conn_01x02_Male, Connector_PinHeader_2.54mm:PinHeader_1x02_P2.54mm_Vertical, F.Cu at (64.0, 124.0)
- added J74: Conn_01x02_Male, Connector_PinHeader_2.54mm:PinHeader_1x02_P2.54mm_Vertical, F.Cu at (65.0, 128.0)
- added J75: Conn_01x02_Male, Connector_PinHeader_2.54mm:PinHeader_1x02_P2.54mm_Vertical, F.Cu at (65.0, 134.0)
- added J76: Conn_01x02_Male, Connector_PinHeader_2.54mm:PinHeader_1x02_P2.54mm_Vertical, F.Cu at (66.0, 139.0)
- added J77: Conn_01x02_Male, Connector_PinHeader_2.54mm:PinHeader_1x02_P2.54mm_Vertical, F.Cu at (66.2, 147.0)
- added J78: Conn_01x02_Male, Connector_PinHeader_2.54mm:PinHeader_1x02_P2.54mm_Vertical, F.Cu at (110.0, 149.0)
- added J79: Conn_01x02_Male, Connector_PinHeader_2.54mm:PinHeader_1x02_P2.54mm_Vertical, F.Cu at (66.2, 143.0)
- added J80: Conn_01x02_Male, Connector_PinHeader_2.54mm:PinHeader_1x02_P2.54mm_Vertical, F.Cu at (114.2, 142.2)
- added J81: Conn_01x02_Male, Connector_PinHeader_2.54mm:PinHeader_1x02_P2.54mm_Vertical, F.Cu at (96.0, 129.0)
- added J82: Conn_01x02_Male, Connector_PinHeader_2.54mm:PinHeader_1x02_P2.54mm_Vertical, F.Cu at (95.0, 135.0)
- added J83: Conn_01x02_Male, Connector_PinHeader_2.54mm:PinHeader_1x02_P2.54mm_Vertical, F.Cu at (94.0, 139.0)
- added J84: Conn_01x02_Male, Connector_PinHeader_2.54mm:PinHeader_1x02_P2.54mm_Vertical, F.Cu at (93.0, 153.0)
- added J85: Conn_01x02_Male, Connector_PinHeader_2.54mm:PinHeader_1x02_P2.54mm_Vertical, F.Cu at (114.2, 138.6)
- added J86: Conn_01x02_Male, Connector_PinHeader_2.54mm:PinHeader_1x02_P2.54mm_Vertical, F.Cu at (93.5, 145.0)
- added J87: Conn_01x02_Male, Connector_PinHeader_2.54mm:PinHeader_1x02_P2.54mm_Vertical, F.Cu at (66.5, 151.0)
- added Q19: 2N2219, Package_TO_SOT_THT:TO-39-3, F.Cu at (32.0, 133.0)
- added R75: R, Resistor_SMD:R_1206_3216Metric_Pad1.42x1.75mm_HandSolder, F.Cu at (60.5, 173.3)
- moved U1 146.6 mm to (81.0, 142.0)
Connections:
- J70 pad 2: (no net) -> /ICMB1
- J70 pad 3: (no net) -> /GND1
- J71 pad 1: (no net) -> Net-(J71-Pad1)
- J71 pad 30: (no net) -> Net-(J71-Pad30)
- J71 pad 31: (no net) -> Net-(J71-Pad31)
- J71 pad 32: (no net) -> Net-(J71-Pad32)
- J71 pad 33: (no net) -> Net-(J71-Pad33)
- J71 pad 34: (no net) -> Net-(J71-Pad34)
- J71 pad 35: (no net) -> Net-(J71-Pad35)
- J71 pad 36: (no net) -> Net-(J71-Pad36)
- J71 pad 37: (no net) -> Net-(J71-Pad37)
- J71 pad 38: (no net) -> Net-(J71-Pad38)
- J71 pad 39: (no net) -> Net-(J71-Pad39)
- J71 pad 40: (no net) -> Net-(J71-Pad40)
- U1 pad 1: Net-(U1-Pad1) -> /EN
- U1 pad 13: Net-(U1-Pad13) -> /SLOW
